File: PayloadPCBFLIGHT/PayloadPCBFLIGHT.kicad_sch (KiCad schematic)
At the start: 16 parts, among them IC1 TPS610333DRLR, J1 Conn_01x06_Socket, J2 Conn_01x06_Socket, J3 Conn_01x06_Socket, J4 Conn_01x06_Socket, J5 Conn_01x02_Pin, U1 LM3281YFQR, U2 DRV8835DSSR, U3 DRV8835DSSR, U4 ESP32-S3-WROOM-1

Commit message: hi
Parts:
- removed IC1: TPS610333DRLR, SOTFL50P160X60-8N, symbol TPS610333DRLR:TPS610333DRLR
- removed U1: LM3281YFQR, LM3281YFQR:BGA6N40P2X3_116X143X67N, symbol LM3281YFQR:LM3281YFQR
- added C5: 100nF, symbol Device:C
- added C6: 22uF, symbol Device:C
- added U1: AP63203WU-7, AP63203WU-7_DIO, symbol 2025-09-22_22-02-52:AP63203WU-7
- added U5: AP63205WU-7, SOIC_05WU-7_DIO, symbol 2025-09-22_21-52-11:AP63205WU-7
- C1: value 2.2uF -> 10uF
- C2: value 2.2uF -> 22uF
- C3: value 4.7uF -> 10uF
- C4: value 10uF -> 100nF
- L1, L2: value .47uH -> 4.7uH
Connections:
- net +3.3V is gone; now on net +5V: C2.1, L1.2
- net +5V: now also L2.2, C6.1, U1.1 (FB), U5.1 (FB); no longer C4.1
- net GND: now also C6.2, U1.4 (GND), U5.4 (GND); no longer C4.2
- net at C1.2, C3.2, J5.1 (Pin_1): now also U1.2 (EN), U1.3 (VIN), U5.2 (EN), U5.3 (VIN)
- net at L1.1: now also C5.1, U5.5 (SW)
- net at L2.1: now also C4.1, U1.5 (SW)
- new net: C4.2, U1.6 (BST)
- new net: C5.2, U5.6 (BST)
Other:
- note added: "7-8.4 bATTERY"
- moved on the sheet: C1, C2, J1, J2, J3, J4, J5, L1, U2, U3, U4
